File: 555.kicad_pcb (KiCad board)
At the start: 2 copper layers, 120 x 35 mm, 62 parts, among them J2 Screw_Terminal_01x02, P1 USB_C_Plug, SW1 SW_Push, SW2 SW_Push, SW3 SW_Push, SW4 SW_Push, SW5 SW_Push, SW6 SW_Push, SW7 SW_Push, SW8 SW_Push, U1 NE555P

Commit message: marked
Other:
- board text added: "PTR 2022"
Changed lines of the file:
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@@
     (pts
       (xy 84.5 89.25)
+      (xy 65.25 87)
       (xy 56.25 89.25)
       (xy 53 84.75)
@@
   (gr_line (start 75.087651 77) (end 78.087651 77) (layer "F.SilkS") (width 0.15))
   (gr_line (start 77 83) (end 77 82) (layer "F.SilkS") (width 0.15))
+  (gr_poly
+    (pts
+      (xy 84.5 89.75)
+      (xy 56.5 89.5)
+      (xy 65.25 87.5)
+    ) (layer "F.Mask") (width 0.15) (fill solid))
   (gr_line (start 31 92) (end 151 92) (layer "Edge.Cuts") (width 0.1))
   (gr_line (start 151 57) (end 31 57) (layer "Edge.Cuts") (width 0.1))
@@
     (effects (font (size 1.5 1.5) (thickness 0.3) italic))
   )
+  (gr_text "PTR 2022" (at 37.5 90.25 -180) (layer "B.Mask")
+    (effects (font (size 1 1) (thickness 0.15)) (justify mirror))
+  )
+  (gr_text "PTR 2022" (at 37.5 90.25) (layer "F.Mask")
+    (effects (font (size 1 1) (thickness 0.15)))
+  )
   (segment (start 142.955 79.325) (end 142.955 78.345) (width 0.5) (layer "F.Cu") (net 1))
